File: Circuit/Mouse-Control-Circuit.kicad_pcb (KiCad board)
At the start: 2 copper layers, 21 parts, among them U1 TL074

Commit message: Jumpers
Parts:
- added C10: 330n, Capacitor_THT:C_Rect_L7.0mm_W3.5mm_P5.00mm, F.Cu at (72.2, 96.3)
- added C11: 330n, Capacitor_THT:C_Rect_L7.0mm_W3.5mm_P5.00mm, F.Cu at (72.2, 101.4)
- added C7: 1u, Capacitor_THT:C_Rect_L7.0mm_W3.5mm_P5.00mm, F.Cu at (72.2, 81.2)
- added C8: 100n, Capacitor_THT:C_Rect_L7.0mm_W3.5mm_P5.00mm, F.Cu at (72.2, 86.2)
- added C9: 100n, Capacitor_THT:C_Rect_L7.0mm_W3.5mm_P5.00mm, F.Cu at (72.2, 91.3)
- added D5: 1N4148, Diode_THT:D_DO-35_SOD27_P7.62mm_Horizontal, F.Cu at (58.7, 125.0)
- added D6: 1N4148, Diode_THT:D_DO-35_SOD27_P7.62mm_Horizontal, F.Cu at (58.7, 128.6)
- added D7: 1N4148, Resistor_THT:R_Axial_DIN0207_L6.3mm_D2.5mm_P10.16mm_Horizontal, F.Cu at (58.7, 80.7)
- added J1: Screw_Terminal_01x02, TerminalBlock:TerminalBlock_Altech_AK300-2_P5.00mm, F.Cu at (129.3, 123.2)
- added J2: Screw_Terminal_01x02, TerminalBlock:TerminalBlock_Altech_AK300-2_P5.00mm, F.Cu at (140.7, 123.2)
- added L3: 10u, Resistor_THT:R_Axial_DIN0207_L6.3mm_D2.5mm_P10.16mm_Horizontal, F.Cu at (58.7, 92.8)
- added M1: Motor_DC, Resistor_THT:R_Axial_DIN0207_L6.3mm_D2.5mm_P10.16mm_Horizontal, F.Cu at (58.7, 96.9)
- added M2: Motor_DC, Resistor_THT:R_Axial_DIN0207_L6.3mm_D2.5mm_P10.16mm_Horizontal, F.Cu at (58.7, 101.0)
- added Q1: TIP120, Package_TO_SOT_THT:TO-220-3_Vertical, F.Cu at (73.7, 107.8)
- added Q2: TIP120, Package_TO_SOT_THT:TO-220-3_Vertical, F.Cu at (73.7, 113.8)
- added Q3: NMOS, Package_TO_SOT_THT:TO-220-3_Vertical, F.Cu at (73.7, 119.8)
- added R10: 100, Resistor_THT:R_Axial_DIN0207_L6.3mm_D2.5mm_P10.16mm_Horizontal, F.Cu at (58.7, 113.1)
- added R12: 1M, Resistor_THT:R_Axial_DIN0207_L6.3mm_D2.5mm_P10.16mm_Horizontal, F.Cu at (58.7, 117.2)
- added R13: 500k, Resistor_THT:R_Axial_DIN0207_L6.3mm_D2.5mm_P10.16mm_Horizontal, F.Cu at (58.7, 121.2)
- added R4: 100, Resistor_THT:R_Axial_DIN0207_L6.3mm_D2.5mm_P10.16mm_Horizontal, F.Cu at (58.7, 105.0)
- added R9: 100, Resistor_THT:R_Axial_DIN0207_L6.3mm_D2.5mm_P10.16mm_Horizontal, F.Cu at (58.7, 109.0)
- added U2: Pico, MCU_RaspberryPi_and_Boards:RPi_Pico_SMD_TH, F.Cu at (45.1, 105.2)
- added U3: uA7805, Package_TO_SOT_THT:TO-220-3_Vertical, F.Cu at (73.7, 125.7)
Routing:
- net GND: track 81.1 -> 120.5 mm
- net VCC: track 0.00 -> 19.8 mm
- net VEE: track 0.00 -> 18.0 mm
- added copper zone on B.Cu, net GND
- removed copper zone on B.Cu, net (none)

Commit message: PCB
Parts:
- removed C7: 1u, Capacitor_THT:C_Rect_L7.0mm_W3.5mm_P5.00mm
- removed C8, C9: 100n, Capacitor_THT:C_Rect_L7.0mm_W3.5mm_P5.00mm
- removed D5, D6: 1N4148, Diode_THT:D_DO-35_SOD27_P7.62mm_Horizontal
- removed D7: 1N4148, Resistor_THT:R_Axial_DIN0207_L6.3mm_D2.5mm_P10.16mm_Horizontal
- removed L3: 10u, Resistor_THT:R_Axial_DIN0207_L6.3mm_D2.5mm_P10.16mm_Horizontal
- removed Q3: NMOS, Package_TO_SOT_THT:TO-220-3_Vertical
- removed R10: 100, Resistor_THT:R_Axial_DIN0207_L6.3mm_D2.5mm_P10.16mm_Horizontal
- removed R12: 1M, Resistor_THT:R_Axial_DIN0207_L6.3mm_D2.5mm_P10.16mm_Horizontal
- removed R13: 500k, Resistor_THT:R_Axial_DIN0207_L6.3mm_D2.5mm_P10.16mm_Horizontal
- removed R2, R5: 15k, Resistor_THT:R_Axial_DIN0207_L6.3mm_D2.5mm_P10.16mm_Horizontal
- removed R7, R8: 10k, Resistor_THT:R_Axial_DIN0207_L6.3mm_D2.5mm_P10.16mm_Horizontal
- added H1: MountingHole, MountingHole:MountingHole_3.2mm_M3, F.Cu at (99.2, 54.5)
- added H2: MountingHole, MountingHole:MountingHole_3.2mm_M3, F.Cu at (176.8, 54.5)
- added H3: MountingHole, MountingHole:MountingHole_3.2mm_M3, F.Cu at (99.2, 143.5)
- added H4: MountingHole, MountingHole:MountingHole_3.2mm_M3, F.Cu at (176.8, 143.5)
- added RV1: R_Potentiometer, Potentiometer_THT:Potentiometer_Vishay_T73YP_Vertical, F.Cu at (125.7, 76.2)
- added RV2: R_Potentiometer, Potentiometer_THT:Potentiometer_Vishay_T73YP_Vertical, F.Cu at (145.9, 76.2)
- M1, M2: footprint Resistor_THT:R_Axial_DIN0207_L6.3mm_D2.5mm_P10.16mm_Horizontal -> TerminalBlock:TerminalBlock_Altech_AK300-2_P5.00mm
- R3, R6: moved to F.Cu
- moved R9 105.6 mm to (163.2, 124.4), turned to -90 degrees
- moved M2 91.8 mm to (144.8, 133.0), turned to 180 degrees
- moved U2 90.8 mm to (135.9, 106.7), turned to 90 degrees
- moved Q2 88.8 mm to (160.0, 134.5), turned to 90 degrees
- moved M1 79.7 mm to (129.8, 133.0), turned to 180 degrees
- moved J2 51.4 mm to (99.0, 93.2), turned to -90 degrees
- moved R4 51.3 mm to (106.7, 123.1), turned to -90 degrees
- moved U3 49.9 mm to (101.0, 84.0)
- moved Q1 45.8 mm to (111.8, 133.3), turned to 90 degrees
- moved C11 42.4 mm to (107.5, 78.0), turned to 180 degrees
- moved J1 33.2 mm to (99.0, 109.8), turned to 90 degrees
- moved C10 28.5 mm to (99.5, 88.0)
- moved R3 28.2 mm to (116.8, 73.7)
- moved R6 28.0 mm to (154.9, 73.7)
- moved D1 26.5 mm to (119.5, 70.8)
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Connections:
- C10 pad 1: VCC -> +9V
- J2 pad 1: VEE -> +9V
- J2 pad 2: unconnected-(J2-Pin_2-Pad2) -> -9V
- U1 pad 11: VEE -> -9V
- U1 pad 4: VCC -> +9V
- U2 pad 19: unconnected-(U2-GPIO14-Pad19) -> /MOTOR_PWM_R
- U2 pad 2: /MOTOR_PWM_R -> unconnected-(U2-GPIO1-Pad2)
- U2 pad 31: /SENSOR_IN_R -> /PEAK_OUT_R
- U2 pad 32: /SENSOR_IN_L -> /PEAK_OUT_L
- U2 pad 4: /BOOST_CONVERTER_PWM -> unconnected-(U2-GPIO2-Pad4)
- U3 pad 1: VCC -> +9V
Routing:
- net GND: track 120.5 -> 0.00 mm
- net -9V: track 0.00 -> 101.5 mm
- net +9V: track 0.00 -> 89.1 mm
- net VCC: track 19.8 -> 84.2 mm
- net Net-(M2--): track 0.00 -> 26.4 mm
- net +5V: track 0.00 -> 23.8 mm
- net VEE: track 18.0 -> 0.00 mm
- net Net-(M1--): track 0.00 -> 13.9 mm
- net /MOTOR_PWM_R: track 0.00 -> 11.2 mm
- net /MOTOR_PWM_L: track 0.00 -> 9.64 mm
- net /PEAK_OUT_R: track 10.1 -> 17.0 mm
- net Net-(D2-K): track 9.95 -> 16.4 mm
- net Net-(Q1-B): track 0.00 -> 5.08 mm
- net Net-(D4-K): track 9.93 -> 14.1 mm
- net Net-(U1A--): track 5.09 -> 9.25 mm
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- added copper zone on F.Cu, net GND
- removed copper zone on B.Cu, net GND
Other:
- board outline added: 100 x 100 mm
